Commit message: add: 移动机器人相关研究

File: robot_control_ros2/src/simple_arm_description/urdf/simple_2dof_arm.urdf (robot description, URDF)
Before this commit: robot simple_2dof_arm, 3 links, 2 joints
Links:
- added link tool0, mass 0.05; collision sphere radius=0.04; visual sphere radius=0.04
- link base_link: mass None -> 1.0
- link link1: mass None -> 0.5
- link link2: mass None -> 0.4
Joints:
- added joint tool0_fixed_joint: type fixed, parent link2, child tool0, origin xyz=0.8 0 0 rpy=0 0 0

File: robot_control_ros2/src/simple_arm_description/urdf/simple_2dof_arm.urdf.xacro (robot description, xacro)
@@ -1,105 +1,5 @@
 <?xml version="1.0"?>
 <robot name="simple_2dof_arm" xmlns:xacro="http://www.ros.org/wiki/xacro">
-  <!-- ===================== -->
-  <!-- Parameters -->
-  <!-- ===================== -->
-  <xacro:property name="base_size_x" value="0.25"/>
-  <xacro:property name="base_size_y" value="0.25"/>
-  <xacro:property name="base_size_z" value="0.10"/>
-  <xacro:property name="link1_length" value="1.0"/>
-  <xacro:property name="link2_length" value="0.8"/>
-  <xacro:property name="link1_width" value="0.08"/>
-  <xacro:property name="link2_width" value="0.06"/>
-  <!-- ===================== -->
-  <!-- Materials -->
-  <!-- ===================== -->
-  <material name="gray">
-    <color rgba="0.5 0.5 0.5 1.0"/>
-  </material>
-  <material name="blue">
-    <color rgba="0.1 0.3 0.9 1.0"/>
-  </material>
-  <material name="green">
-    <color rgba="0.1 0.8 0.2 1.0"/>
-  </material>
-<!-- ===================== -->
-<!-- base_link -->
-<!-- ===================== -->
-<link name="base_link">
-  <visual>
-    <origin xyz="0 0 0" rpy="0 0 0"/>
-    <geometry>
-      <box size="${base_size_x} ${base_size_y} ${base_size_z}"/>
-    </geometry>
-    <material name="gray"/>
-  </visual>
-  <collision>
-    <origin xyz="0 0 0" rpy="0 0 0"/>
-    <geometry>
-      <box size="${base_size_x} ${base_size_y} ${base_size_z}"/>
-    </geometry>
-  </collision>
-</link>
-  <!-- ===================== -->
-  <!-- joint1: base_link -> link1 -->
-  <!-- ===================== -->
-  <joint name="joint1" type="revolute">
-    <parent link="base_link"/>
-    <child link="link1"/>
-    <!-- joint1 位于 base_link 上方一点 -->
-    <origin xyz="0 0 ${base_size_z / 2.0}" rpy="0 0 0"/>
-    <!-- 绕 z 轴旋转 -->
-    <axis xyz="0 0 1"/>
-    <limit lower="-3.14" upper="3.14" effort="10.0" velocity="1.0"/>
-  </joint>
-<!-- ===================== -->
-<!-- link1 -->
-<!-- ===================== -->
-<link name="link1">
-  <visual>
-    <!-- link1 的坐标系在 joint1 处，所以盒子的中心放在 x=0.5 处 -->
-    <origin xyz="${link1_length / 2.0} 0 0" rpy="0 0 0"/>
-    <geometry>
-      <box size="${link1_length} ${link1_width} ${link1_width}"/>
-    </geometry>
-    <material name="blue"/>
-  </visual>
-  <collision>
-    <origin xyz="${link1_length / 2.0} 0 0" rpy="0 0 0"/>
-    <geometry>
-      <box size="${link1_length} ${link1_width} ${link1_width}"/>
-    </geometry>
-  </collision>
-</link>
-  <!-- ===================== -->
-  <!-- joint2: link1 -> link2 -->
-  <!-- ===================== -->
-  <joint name="joint2" type="revolute">
-    <parent link="link1"/>
-    <child link="link2"/>
-    <!-- joint2 位于 link1 末端 -->
-    <origin xyz="${link1_length} 0 0" rpy="0 0 0"/>
-    <!-- 绕 z 轴旋转 -->
-    <axis xyz="0 0 1"/>
-    <limit lower="-1.57" upper="1.57" effort="10.0" velocity="1.0"/>
-  </joint>
-<!-- ===================== -->
-<!-- link2 -->
-<!-- ===================== -->
-<link name="link2">
-  <visual>
-    <!-- link2 的坐标系在 joint2 处，所以盒子的中心放在 x=0.4 处 -->
-    <origin xyz="${link2_length / 2.0} 0 0" rpy="0 0 0"/>
-    <geometry>
-      <box size="${link2_length} ${link2_width} ${link2_width}"/>
-    </geometry>
-    <material name="green"/>
-  </visual>
-  <collision>
-    <origin xyz="${link2_length / 2.0} 0 0" rpy="0 0 0"/>
-    <geometry>
-      <box size="${link2_length} ${link2_width} ${link2_width}"/>
-    </geometry>
-  </collision>
-</link>
+  <xacro:include filename="$(find simple_arm_description)/urdf/simple_2dof_arm_model.xacro"/>
+  <xacro:simple_2dof_arm_model/>
 </robot>

File: robot_control_ros2/src/simple_arm_moveit_config/config/simple_2dof_arm.ros2_control.xacro (robot description, xacro)
@@ -1,10 +1,14 @@
 <?xml version="1.0"?>
 <robot xmlns:xacro="http://www.ros.org/wiki/xacro">
-    <xacro:macro name="simple_2dof_arm_ros2_control" params="name initial_positions_file">
+    <xacro:macro name="simple_2dof_arm_ros2_control" params="name initial_positions_file hardware_type:=fake ros2_controllers_file:=''">
         <xacro:property name="initial_positions" value="${xacro.load_yaml(initial_positions_file)['initial_positions']}"/>
         <ros2_control name="${name}" type="system">
             <hardware>
-                <!-- By default, set up controllers for simulation. This won't work on real hardware -->
-                <plugin>mock_components/GenericSystem</plugin>
+                <xacro:if value="${hardware_type == 'fake'}">
+                    <plugin>mock_components/GenericSystem</plugin>
+                </xacro:if>
+                <xacro:if value="${hardware_type == 'gazebo'}">
+                    <plugin>gz_ros2_control/GazeboSimSystem</plugin>
+                </xacro:if>
             </hardware>
             <joint name="joint1">
@@ -23,4 +27,11 @@
             </joint>
         </ros2_control>
+        <xacro:if value="${hardware_type == 'gazebo'}">
+            <gazebo>
+                <plugin filename="gz_ros2_control-system" name="gz_ros2_control::GazeboSimROS2ControlPlugin">
+                    <parameters>${ros2_controllers_file}</parameters>
+                </plugin>
+            </gazebo>
+        </xacro:if>
     </xacro:macro>
 </robot>

File: robot_control_ros2/src/simple_arm_moveit_config/config/simple_2dof_arm.urdf.xacro (robot description, xacro)
@@ -2,8 +2,16 @@
 <robot xmlns:xacro="http://www.ros.org/wiki/xacro" name="simple_2dof_arm">
     <xacro:arg name="initial_positions_file" default="initial_positions.yaml" />
-    <!-- Import simple_2dof_arm urdf file -->
-    <xacro:include filename="$(find simple_arm_description)/urdf/simple_2dof_arm.urdf" />
+    <xacro:arg name="hardware_type" default="fake" />
+    <xacro:arg name="ros2_controllers_file" default="" />
+    <xacro:arg name="use_world_joint" default="false" />
+    <!-- Import and instantiate the robot model. -->
+    <xacro:include filename="$(find simple_arm_description)/urdf/simple_2dof_arm_model.xacro" />
+    <xacro:simple_2dof_arm_model use_world_joint="$(arg use_world_joint)"/>
     <!-- Import control_xacro -->
     <xacro:include filename="simple_2dof_arm.ros2_control.xacro" />
-    <xacro:simple_2dof_arm_ros2_control name="FakeSystem" initial_positions_file="$(arg initial_positions_file)"/>
+    <xacro:simple_2dof_arm_ros2_control
+        name="SimpleArmSystem"
+        initial_positions_file="$(arg initial_positions_file)"
+        hardware_type="$(arg hardware_type)"
+        ros2_controllers_file="$(arg ros2_controllers_file)"/>
 </robot>
