Commit message: add: aubo_i5 修改urdf 增加moveit_config

File: aubo_i5_ros2_control/src/robot_description/urdf/arm.xacro (robot description, xacro)
@@ -283,61 +283,3 @@
     <limit lower="-3.04" upper="3.04" effort="300" velocity="100" />
   </joint>
-  <!-- /////////////////////////////////   i5 pedestal_Link   //////////////////////////////////////
-  <link name="pedestal_Link">
-    <visual>
-      <geometry>
-        <mesh filename="package://aubo_description/meshes/aubo_i5/collision/pedestal.STL" />
-      </geometry>
-    </visual>
-  </link>
-  <joint name="pedestal_joint" type="fixed">
-    <parent link="pedestal_Link"/>
-    <child link="base_link"/>
-    <origin xyz="0.0 0.0 0.402" rpy="0.0 0.0 0.0" />
-  </joint>
--->
- <!-- /////////////////////////////////   world   ////////////////////////////////////// -->
-  <link name="world" />
-  <joint name="world_joint" type="fixed">
-    <parent link="world" />
-    <child link ="base_link" />
-    <origin xyz="0.0 0.0 0.0" rpy="0.0 0.0 0.0" />
-  </joint>
- <!-- /////////////////////////////////   jawasm1   //////////////////////////////////////
-  <xacro:robotiq_85_gripper prefix="" parent="tool" >
-	<origin xyz="0 0 0" rpy="0 ${-M_PI/2} 0"
-  </xacro:robotiq_85_gripper>
-  <xacro:include filename="(find aubo_description)/urdf/jawasm1.urdf"/>-->
-  <!-- /////////////////////////////////   gazebo color   ////////////////////////////////////// -->
-  <!--<gazebo reference="pedestal_Link">
-     <material>Gazebo/Grey</material>
-  </gazebo>-->
-  <!--////////////////////////////////// Transmissions for ROS Control //////////////////////////-->
-<xacro:macro name="aubo_arm_transmission" params="joint_name">
-     <transmission name="${joint_name}_trans">
-       <type>transmission_interface/SimpleTransmission</type>
-       <joint name="${joint_name}">
-         <!--<hardwareInterface>hardware_interface/PositionJointInterface</hardwareInterface>-->
-         <hardwareInterface>hardware_interface/PositionJointInterface</hardwareInterface>
-       </joint>
-       <actuator name="${joint_name}_motor">
-	 <hardwareInterface>hardware_interface/PositionJointInterface</hardwareInterface>
-         <mechanicalReduction>1</mechanicalReduction>
-       </actuator>
-     </transmission>
- </xacro:macro>
-  <xacro:aubo_arm_transmission joint_name="shoulder_joint"/>
-  <xacro:aubo_arm_transmission joint_name="upperArm_joint"/>
-  <xacro:aubo_arm_transmission joint_name="foreArm_joint"/>
-  <xacro:aubo_arm_transmission joint_name="wrist1_joint"/>
-  <xacro:aubo_arm_transmission joint_name="wrist2_joint"/>
-  <xacro:aubo_arm_transmission joint_name="wrist3_joint"/>
-  <!-- ros_control plugin -->
-  <gazebo>
-      <plugin name="gazebo_ros_control" filename="libgazebo_ros_control.so">
-          <robotNamespace>/aubo_i5</robotNamespace>
-	  <robotSimType>gazebo_ros_control/DefaultRobotHWSim</robotSimType>
-          <legacyModeNS>true</legacyModeNS>
-      </plugin>
-  </gazebo>
 </robot>

File: aubo_i5_ros2_control/src/robot_description/urdf/aubo_i5.xacro (robot description, xacro)
@@ -9,4 +9,6 @@
         <child  link="gripper_base_link" />
     </joint>
+     <!-- /////////////////////////////////   world   ////////////////////////////////////// -->
+    <link name="world" />
     <joint name="world2base_link" type="fixed">
         <origin xyz="0 0 0" rpy="0 0 0 " />

Commit message: fix: 修改模型惯性矩阵

File: aubo_i5_ros2_control/src/robot_description/urdf/arm.xacro (robot description, xacro)
@@ -32,13 +32,13 @@
     </xacro:macro>
     <xacro:macro name="I5_UpperArm_Inertia">
-        <origin xyz="0.304 0.0 -0.03"
-                rpy="0 0 0" />
-        <mass value="11.90" />
-        <inertia ixx="0.0305"
-                 ixy="0"
-                 ixz="0"
-                 iyy="0.4505"
+        <origin xyz="0.2040 0.0 0.006603"
+                rpy="0 0 0" />
+        <mass value="10.836261" />
+        <inertia ixx="0.026024"
+                 ixy="0.00002"
+                 ixz="0"
+                 iyy="0.432805"
                  iyz="0"
-                 izz="0.0095" />
+                 izz="0.425155" />
     </xacro:macro>
     <xacro:macro name="I5_ForeArm_Inertia">

File: aubo_i5_ros2_control/src/robot_description/urdf/aubo_i5_arm.urdf (robot description, URDF)
Before this commit: robot aubo_i5, 12 links, 11 joints
Links:
- link upperArm_Link: mass 11.90 -> 10.836261
