Commit message: fix: gripper joint

File: aubo_i5_ros2_control/src/aubo_i5_moveit_config/config/aubo_i5.urdf.xacro (robot description, xacro)
@@ -5,5 +5,5 @@
     <xacro:arg name="initial_positions_file" default="initial_positions.yaml" />
     <!-- Import aubo_i5 urdf file 机器人模型文件 -->
-    <xacro:include filename="$(find robot_description)/urdf/aubo_i5_arm.urdf" />
+    <xacro:include filename="$(find robot_description)/urdf/aubo_i5.xacro" />
     <!-- Import control_xacro -->
     <xacro:include filename="aubo_i5.ros2_control.xacro" />

File: aubo_i5_ros2_control/src/robot_description/urdf/jiazhua.urdf (robot description, URDF)
Before this commit: robot jiazhua, 4 links, 3 joints
Joints:
- joint joint1: type continuous -> fixed
- joint joint2: type continuous -> fixed
