Commit message: add: auboi5 gazebo部分 但存在错误(world+base_link)

File: aubo_i5_ros2_control/src/aubo_i5_moveit_config/config/aubo_i5.ros2_control.xacro (robot description, xacro)
@@ -1,5 +1,5 @@
 <?xml version="1.0"?>
 <robot xmlns:xacro="http://www.ros.org/wiki/xacro">
-    <xacro:macro name="aubo_i5_ros2_control" params="name initial_positions_file">
+    <xacro:macro name="aubo_i5_ros2_control" params="name initial_positions_file hardware_type ros2_controllers_file">
         <xacro:property name="initial_positions" value="${xacro.load_yaml(initial_positions_file)['initial_positions']}"/>
         <ros2_control name="${name}" type="system">

File: aubo_i5_ros2_control/src/aubo_i5_moveit_config/config/aubo_i5.urdf.xacro (robot description, xacro)
@@ -8,4 +8,5 @@
     <!-- Import control_xacro -->
     <xacro:include filename="aubo_i5.ros2_control.xacro" />
-    <xacro:aubo_i5_ros2_control name="FakeSystem" initial_positions_file="$(arg initial_positions_file)"/>
+    <xacro:aubo_i5_ros2_control name="control_system" initial_positions_file="$(arg initial_positions_file)"
+        hardware_type="$(arg hardware_type)" ros2_controllers_file="$(arg ros2_controllers_file)"/>
 </robot>

Commit message: add: aubo i5 hardware

File: aubo_i5_ros2_control/src/aubo_i5_moveit_config/config/aubo_i5.ros2_control.xacro (robot description, xacro)
@@ -1,5 +1,6 @@
 <?xml version="1.0"?>
 <robot xmlns:xacro="http://www.ros.org/wiki/xacro">
-    <xacro:macro name="aubo_i5_ros2_control" params="name initial_positions_file hardware_type ros2_controllers_file">
+    <xacro:macro name="aubo_i5_ros2_control" params="name initial_positions_file hardware_type ros2_controllers_file
+        robot_ip enable_motion">
         <xacro:property name="initial_positions" value="${xacro.load_yaml(initial_positions_file)['initial_positions']}"/>
         <ros2_control name="${name}" type="system">
@@ -10,4 +11,13 @@
                 <xacro:if value="${hardware_type == 'gazebo'}">
                     <plugin>gz_ros2_control/GazeboSimSystem</plugin>
+                </xacro:if>
+                <xacro:if value="${hardware_type == 'real'}">
+                    <plugin>aubo_i5_hardware/AuboI5System</plugin>
+                    <param name="robot_ip">$(arg robot_ip)</param>
+                    <param name="rpc_port">30004</param>
+                    <param name="rtde_port">30010</param>
+                    <param name="connect_timeout_ms">1000</param>
+                    <param name="command_timeout_ms">100</param>
+                    <param name="enable_motion">$(arg enable_motion)</param>
                 </xacro:if>
                 <!-- By default, set up controllers for simulation. This won't work on real hardware -->

File: aubo_i5_ros2_control/src/aubo_i5_moveit_config/config/aubo_i5.urdf.xacro (robot description, xacro)
@@ -4,4 +4,6 @@
     <xacro:arg name="ros2_controllers_file" default="ros2_controllers.yaml"/>
     <xacro:arg name="initial_positions_file" default="initial_positions.yaml" />
+    <xacro:arg name="robot_ip" default="192.168.1.2"/>
+    <xacro:arg name="enable_motion" default="false"/>
     <!-- Import aubo_i5 urdf file 机器人模型文件 -->
     <xacro:include filename="$(find robot_description)/urdf/aubo_i5.xacro" />
@@ -9,4 +11,5 @@
     <xacro:include filename="aubo_i5.ros2_control.xacro" />
     <xacro:aubo_i5_ros2_control name="control_system" initial_positions_file="$(arg initial_positions_file)"
-        hardware_type="$(arg hardware_type)" ros2_controllers_file="$(arg ros2_controllers_file)"/>
+        hardware_type="$(arg hardware_type)" ros2_controllers_file="$(arg ros2_controllers_file)"
+        robot_ip="$(arg robot_ip)" enable_motion="$(arg enable_motion)"/>
 </robot>
